Commit message: se agrega camara al simulador

File: src/kobuki/kobuki_description/urdf/kobuki.urdf.xacro (robot description, xacro)
@@ -1,3 +1,5 @@
 <?xml version="1.0" ?>
+<sdf version='1.6'>
+  <world name='kobuki_empty_world'>
 <!--
   This is not a standalone urdf for kobuki. It simply defines the 'kobuki' tag that can
@@ -9,4 +11,5 @@
   <xacro:include filename="$(find kobuki_description)/urdf/common_properties.urdf.xacro"/>
   <xacro:include filename="$(find kobuki_description)/urdf/kobuki_gazebo.urdf.xacro"/>
+  <xacro:property name="camara" value="0.05" />
   <!-- Kobuki -->
   <xacro:macro name="kobuki">
@@ -209,4 +212,39 @@
     </link>
     <!-- kobuki agrega link_palo y base-->
+!--
+    <!--link name="camara">
+      <visual>
+        <geometry>
+          <cylinder length="0.1" radius="0.1"/>
+        </geometry>
+        <origin xyz="0 1.50 0" rpy="0 0 0"/>
+      </visual>
+    </link-->
+    <joint name="camara_joint" type="fixed">
+      <axis xyz="0 1 0" />
+      <origin xyz="0 0 0.8" rpy="0 0 0"/>
+      <parent link="link_palo"/>
+      <child link="camara"/>
+    </joint>
+    <link name="camara">
+      <!--collision>
+        <origin xyz="0 0 0" rpy="0 0 0"/>
+        <geometry>
+      <box size="${camara ${camara} ${camara}"/>
+        </geometry>
+      </collision-->
+      <visual>
+        <origin xyz="0 0 0" rpy="0 0 0"/>
+        <geometry>
+      <box size="${camara} ${camara} ${camara}"/>
+        </geometry>
+        <material name="red"/>
+      </visual>
+      <!--inertial>
+        <mass value="1e-5" />
+        <origin xyz="0 0 0" rpy="0 0 0"/>
+        <inertia ixx="1e-6" ixy="0" ixz="0" iyy="1e-6" iyz="0" izz="1e-6" />
+      </inertial-->
+    </link>
     <link name="link_palo" type="fixed">
       <visual>
@@ -229,2 +267,4 @@
   </xacro:macro>
 </robot>
+</world>
+</sdf>

File: src/kobuki/kobuki_description/urdf/kobuki_gazebo.urdf.xacro (robot description, xacro)
@@ -48,4 +48,42 @@
     <gazebo reference="link_palo">
       <material>Gazebo/Black</material>
+    </gazebo>
+    <!-- camara rql-->
+    <gazebo reference="camara">
+      <material>Gazebo/Black</material>
+      <sensor type="camera" name="camara_1">
+        <update_rate>30</update_rate>
+        <camera name="head">
+          <horizontal_fov>1.396234</horizontal_fov>
+          <image>
+            <width>800</width>
+            <height>800</height>
+            <format>R8G8B8</format>
+          </image>
+          <clip>
+            <near>0.02</near>
+            <far>300</far>
+          </clip>
+          <noise>
+            <type>gaussian</type>
+            <mean>0.0</mean>
+            <stddev>0.007</stddev>
+          </noise>
+        </camera>
+        <plugin name="camera_controller" filename="libgazebo_ros_camera.so">
+          <alwaysOn>true</alwaysOn>
+          <updateRate>0.0</updateRate>
+          <cameraName>kobuki_sim/camera_1</cameraName>
+          <imageTopicName>image_raw</imageTopicName>
+          <cameraInfoTopicName>camera_info</cameraInfoTopicName>
+          <frameName>camara</frameName>
+          <hackBaseline>0.07</hackBaseline>
+          <distortionK1>0.0</distortionK1>
+          <distortionK2>0.0</distortionK2>
+          <distortionK3>0.0</distortionK3>
+          <distortionT1>0.0</distortionT1>
+          <distortionT2>0.0</distortionT2>
+        </plugin>
+      </sensor>
     </gazebo>
 	  <gazebo reference="cliff_sensor_left_link">

Commit message: se agrega el kine a kobuki

File: src/kobuki/kobuki_description/urdf/kobuki.urdf.xacro (robot description, xacro)
@@ -12,4 +12,5 @@
   <xacro:include filename="$(find kobuki_description)/urdf/kobuki_gazebo.urdf.xacro"/>
   <xacro:property name="camara" value="0.05" />
+  <xacro:property name="M_PI" value="3.1415926535897931" />
   <!-- Kobuki -->
   <xacro:macro name="kobuki">
@@ -212,13 +213,4 @@
     </link>
     <!-- kobuki agrega link_palo y base-->
-!--
-    <!--link name="camara">
-      <visual>
-        <geometry>
-          <cylinder length="0.1" radius="0.1"/>
-        </geometry>
-        <origin xyz="0 1.50 0" rpy="0 0 0"/>
-      </visual>
-    </link-->
     <joint name="camara_joint" type="fixed">
       <axis xyz="0 1 0" />
@@ -227,4 +219,18 @@
       <child link="camara"/>
     </joint>
+    <!--joint camara de profunidad-->
+    <joint name="camara_profundidad_joint" type="fixed">
+      <!--axis xyz="0 1 0" /-->
+      <origin xyz ="0.1 0 0.15" rpy="0 0 0"/>  <!--heght480-640/2-->
+      <parent link="base_link"/>
+      <child link="camara_profundidad"/>
+    </joint>
+    <joint name="camara_profundidad_optical_joint" type="fixed">
+  <origin xyz="0 0 0" rpy="${-M_PI/2} 0 ${-M_PI/2}" />
+  <parent link="camara_profundidad" />
+  <child link="camara_profundidad_optical" />
+</joint>
+<link name="camara_profundidad_optical"/>
+    <!--camara comun y oridinaria-->
     <link name="camara">
       <!--collision>
@@ -237,5 +243,5 @@
         <origin xyz="0 0 0" rpy="0 0 0"/>
         <geometry>
-      <box size="${camara} ${camara} ${camara}"/>
+          <box size="${camara} ${camara} ${camara}"/>
         </geometry>
         <material name="red"/>
@@ -246,4 +252,13 @@
         <inertia ixx="1e-6" ixy="0" ixz="0" iyy="1e-6" iyz="0" izz="1e-6" />
       </inertial-->
+    </link>
+    <!--camara de profunidad, kinetic microsoft-->
+    <link name="camara_profundidad" type="fixed">
+      <visual>
+        <origin xyz="0 0 0" rpy="0 0 0"/>
+        <geometry>
+          <box size="0.1 0.1 0.1"/>
+        </geometry>
+      </visual>
     </link>
     <link name="link_palo" type="fixed">

File: src/kobuki/kobuki_description/urdf/kobuki_gazebo.urdf.xacro (robot description, xacro)
@@ -87,4 +87,47 @@
       </sensor>
     </gazebo>
+    <!-- camra de profunidad-->
+    <gazebo reference="camara_profundidad">
+      <sensor type="depth" name="xbox_kinetic">
+        <always_on>1</always_on>
+        <visualize>true</visualize>
+        <camera>
+            <horizontal_fov>1.047</horizontal_fov>
+            <image>
+              <width>640</width>
+              <height>480</height>
+              <format>R8G8B8</format>
+            </image>
+            <depth_camera>
+            </depth_camera>
+            <clip>
+                <near>0.3</near>
+                <far>2</far>
+            </clip>
+        </camera>
+            <plugin name="kinect_camera_controller" filename="libgazebo_ros_openni_kinect.so">
+            <alwaysOn>true</alwaysOn>
+                <updateRate>500.0</updateRate>
+                <cameraName>xbox_kinetic</cameraName>
+                <frameName>camara_profundidad_optical</frameName>
+            <imageTopicName>rgb/image_raw</imageTopicName>
+            <depthImageTopicName>depth/image_raw</depthImageTopicName>
+            <pointCloudTopicName>depth/points</pointCloudTopicName>
+            <cameraInfoTopicName>rgb/camera_info</cameraInfoTopicName>
+            <depthImageCameraInfoTopicName>depth/camera_info</depthImageCameraInfoTopicName>
+            <pointCloudCutoff>0.4</pointCloudCutoff>
+                <hackBaseline>0.07</hackBaseline>
+                <distortionK1>0.0</distortionK1>
+                <distortionK2>0.0</distortionK2>
+                <distortionK3>0.0</distortionK3>
+                <distortionT1>0.0</distortionT1>
+                <distortionT2>0.0</distortionT2>
+            <CxPrime>0.0</CxPrime>
+            <Cx>0.0</Cx>
+            <Cy>0.0</Cy>
+            <focalLength>0.0</focalLength>
+          </plugin>
+   </sensor>
+ </gazebo>
 	  <gazebo reference="cliff_sensor_left_link">
 	    <sensor type="ray" name="cliff_sensor_left">
